Commit message: left right wheel

File: description/robot_core.xacro (robot description, xacro)
@@ -1,18 +1,24 @@
 <?xml version="1.0"?>
-<robot xmlns:xacro="http://www.ros.org/wiki/xacro">
-      <material name="whitle">
-        <color rgba="1 1 1 1"/>
+<robot xmlns:xacro="http://www.ros.org/wiki/xacro" name="robot">
+<!-- param -->
+      <material name="white">
+          <color rgba="1 1 1 1" />
       </material>
       <material name="orange">
-        <color rgba="1 0.3 0.1 1"/>
+          <color rgba="1 0.3 0.1 1"/>
       </material>
       <material name="blue">
-        <color rgba="0.2 0.2 1 1"/>
+          <color rgba="0.2 0.2 1 1"/>
       </material>
       <material name="black">
-        <color rgba="0 0 0 0"/>
+          <color rgba="0 0 0 1"/>
       </material>
+      <material name="red">
+          <color rgba="1 0 0 1"/>
+      </material>
+      <!-- BASE LINK -->
       <link name="base_link">
       </link>
+    <!-- CHASSIS LINK -->
       <joint name="chsssis_joint" type="fixed">
         <parent link="base_link"/>
@@ -26,5 +32,35 @@
                 <box size="0.3 0.3 0.15"/>
             </geometry>
-            <material name="white">
+            <material name="white"/>
+        </visual>
+      </link>
+<!-- left wheel -->
+      <joint name="left_wheel_joint" type="continuous">
+        <parent link="base_link"/>
+        <child link="left_wheel"/>
+        <origin xyz="0 0.175 0" rpy="-${pi/2} 0 0"/>
+        <axis xyz="0 0 1"/>
+      </joint>
+      <link name="left_wheel">
+        <visual>
+          <geometry>
+            <cylinder radius="0.05" length="0.04"/>
+          </geometry>
+          <material name="blue"/>
+        </visual>
+      </link>
+<!-- right wheel -->
+      <joint name="right_wheel_joint" type="continuous">
+        <parent link="base_link"/>
+        <child link="right_wheel"/>
+        <origin xyz="0 -0.175 0" rpy="${pi/2} 0 0"/>
+        <axis xyz="0 0 -1"/>
+      </joint>
+      <link name="right_wheel">
+        <visual>
+          <geometry>
+            <cylinder radius="0.05" length="0.04"/>
+          </geometry>
+          <material name="blue"/>
         </visual>
       </link>
